File: HSCanT.kicad_pcb (KiCad board)
At the start: 2 copper layers, 50 x 50 mm, 116 parts, among them J1 Header 1.27 4P, J2 CX90M, J3 2601-1102, J4 2601-1102, J5 2601-1102, J6 2601-1102, SW1 TS3425, U1 0524P, U10 TLP172, U11 TCAN1044AVDR-Q1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

Commit message: update: 更新原理图和PCB
Parts:
- added G***: LOGO, LOGO, F.Cu at (94.9, 24.9)
- added JP1: Jumper_2_Open, Jumper:SolderJumper-2_P1.3mm_Open_RoundedPad1.0x1.5mm, F.Cu at (124.1, 39.8)
- added JP2: Jumper_2_Open, Jumper:SolderJumper-2_P1.3mm_Open_RoundedPad1.0x1.5mm, F.Cu at (114.1, 39.8)
- added JP3: Jumper_2_Open, Jumper:SolderJumper-2_P1.3mm_Open_RoundedPad1.0x1.5mm, F.Cu at (105.7, 39.8)
- added JP4: Jumper_2_Open, Jumper:SolderJumper-2_P1.3mm_Open_RoundedPad1.0x1.5mm, F.Cu at (95.7, 39.8)
- added Q1: 2N7002, Package_DFN_QFN:Diodes_DFN1006-3, F.Cu at (121.5, 40.5)
- added Q2: 2N7002, Package_DFN_QFN:Diodes_DFN1006-3, F.Cu at (111.0, 38.3)
- added Q3: 2N7002, Package_DFN_QFN:Diodes_DFN1006-3, F.Cu at (108.9, 38.3)
- added Q4: 2N7002, Package_DFN_QFN:Diodes_DFN1006-3, F.Cu at (98.3, 40.1)
- added TP6: TestPoint, TestPoint:TestPoint_Pad_D1.0mm, B.Cu at (110.0, 33.8)
- added TP7: TestPoint, TestPoint:TestPoint_Pad_D1.0mm, B.Cu at (110.0, 36.3)
- R10, R16, R21: value 1k -> 10k
- R14, R20, R9: value 0R -> 1k
- R15: value 0R -> 10k
- moved R16 8.79 mm to (114.3, 36.6), turned to -90 degrees
- moved R17 6.91 mm to (98.6, 34.1), turned to -90 degrees
- moved R14 6.05 mm to (109.0, 45.1), turned to 0 degrees
- moved R9 5.98 mm to (110.9, 45.1), turned to 180 degrees
- moved R10 4.06 mm to (113.3, 36.6), turned to -90 degrees
- moved R20 2.52 mm to (98.3, 41.2), turned to 0 degrees
- moved R21 2.42 mm to (98.3, 39.0), turned to 180 degrees
- moved R19 2.19 mm to (121.5, 41.7)
- moved R15 1.90 mm to (121.5, 39.4)
- moved R4 0.97 mm to (101.8, 28.8)
- moved C5 0.97 mm to (101.8, 29.7), turned to 0 degrees
- moved R22 0.37 mm to (94.0, 34.1)
- moved C43 0.37 mm to (91.8, 30.7)
- moved C42 0.37 mm to (89.6, 34.1)
- moved U11 0.37 mm to (91.8, 33.3)
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Connections:
- R10 pad 1: Net-(R10-Pad1) -> /CAN1_RES
- R10 pad 2: /CAN1_RES -> GND
- R14 pad 1: +3V3 -> Net-(R14-Pad1)
- R14 pad 2: Net-(R14-Pad2) -> +3V3
- R15 pad 1: +3V3 -> /CAN0_RES
- R15 pad 2: Net-(R15-Pad2) -> GND
- R16 pad 1: Net-(R14-Pad2) -> /CAN2_RES
- R16 pad 2: /CAN2_RES -> GND
- R19 pad 1: Net-(R15-Pad2) -> Net-(R19-Pad1)
- R19 pad 2: /CAN0_RES -> +3V3
- R20 pad 1: +3V3 -> Net-(R20-Pad1)
- R20 pad 2: Net-(R20-Pad2) -> +3V3
- R21 pad 1: Net-(R20-Pad2) -> /CAN3_RES
- R21 pad 2: /CAN3_RES -> GND
- R9 pad 1: +3V3 -> Net-(R9-Pad1)
- R9 pad 2: Net-(R10-Pad1) -> +3V3
- U10 pad 1: Net-(R14-Pad2) -> Net-(R14-Pad1)
- U10 pad 2: GND -> Net-(JP3-A)
- U12 pad 1: Net-(R20-Pad2) -> Net-(R20-Pad1)
- U12 pad 2: GND -> Net-(JP4-A)
- U7 pad 1: GND -> Net-(R9-Pad1)
- U7 pad 2: Net-(R10-Pad1) -> Net-(JP2-A)
- U9 pad 1: Net-(R15-Pad2) -> Net-(R19-Pad1)
- U9 pad 2: GND -> Net-(JP1-A)
- U9 pad 3: Net-(D10-A2) -> Net-(R11-Pad1)
- U9 pad 4: Net-(R11-Pad1) -> Net-(D10-A2)
Routing:
- net +3V3: track 0.00 -> 160.8 mm, vias 0 -> 12
- net +5V: track 0.00 -> 92.9 mm, vias 0 -> 6
- net RGB_VDD: track 0.00 -> 85.8 mm, vias 0 -> 8
- net GND: track 0.00 -> 79.2 mm, vias 0 -> 54
- net VDD_SOC0: track 0.00 -> 47.4 mm, vias 0 -> 6
- net /RGB_T: track 0.00 -> 39.8 mm, vias 0 -> 4
- net /CAN0_RX: track 0.00 -> 34.9 mm, vias 0 -> 2
- net /CAN0_TX: track 0.00 -> 34.0 mm, vias 0 -> 2
- net VBUS: track 0.00 -> 32.8 mm, vias 0 -> 4
- net /CAN3_RES: track 0.00 -> 26.4 mm, vias 0 -> 2
- net /BOOT0: track 0.00 -> 25.3 mm, vias 0 -> 2
- net /CAN3_RX: track 0.00 -> 25.0 mm, vias 0 -> 2
- net /CAN1_TX: track 0.00 -> 24.6 mm, vias 0 -> 2
- net /CAN1_RX: track 0.00 -> 24.2 mm, vias 0 -> 2
- net /CAN3_TX: track 0.00 -> 23.8 mm, vias 0 -> 2
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- added copper zone on B.Cu, net GND
- added copper zone on F.Cu, net GND
Other:
- board text added: "BL"
- board text added: "G"
- board text added: "GND"
- board text added: "TCK"
- board text added: "TDI"
- board text added: "TDO"
- board text added: "TMS"
- board text added: "V"

Commit message: release: v1.1.0
Parts:
- added D14: LED_G, LED_SMD:LED_0603_1608Metric, F.Cu at (94.9, 19.1)
- added G***: LOGO, LOGO, B.Cu at (110.0, 26.6)
- added R23: 5.1k, Resistor_SMD:R_0402_1005Metric, F.Cu at (115.3, 36.6)
Connections:
- D3 pad 4: /RGB_R -> Net-(D3-DIN)
- D8 pad 2: unconnected-(D8-DOUT-Pad2) -> Net-(D3-DIN)
- U2 pad 22: /RGB_R -> unconnected-(U2B-PB13/TMR1.COMP3/URT3.DE/URT3.RTS/I2C3.SCL/SPI2.MOSI/CAN3.STBY/TRGM0.P01/ADC0.IN5/ADC1.IN5/CMP0.INP2/CMP1.INP2-Pad22)
- U2 pad 25: unconnected-(U2B-PB10/TMR0.COMP2/URT2.DE/URT2.RTS/SPI2.CS0/CAN2.STBY/ACMP.COMP0/USB0.PWR/ADC0.IN2/ADC1.IN2/CMP0.INP4/CMP1.INP4-Pad25) -> /SYS
Routing:
- net Net-(D14-A): track 0.00 -> 51.6 mm, vias 0 -> 2
- net Net-(D3-DIN): track 0.00 -> 26.8 mm, vias 0 -> 2
- net /RGB_R: track 22.7 -> 0.00 mm, vias 2 -> 0
- net GND: track 79.2 -> 100.2 mm, vias 54 -> 80
- net /SYS: track 0.00 -> 5.54 mm
- net /CAN0_TX: track 34.0 -> 33.3 mm
- net Net-(D12-A1): track 24.6 -> 24.1 mm
Other:
- copper layers 2 -> 4
- board text added: "SYS"
- board text added: "V1.1.0"
