File: HSCanT.kicad_sch (KiCad schematic)
At the start: 112 parts, among them J1 Header 1.27 4P, J2 CX90M, J3 2601-1102, J4 2601-1102, J5 2601-1102, J6 2601-1102, SW1 TS3425, U1 0524P, U10 TLP172, U11 TCAN1044AVDR-Q1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

Commit message: update: 更新原理图和PCB
Parts:
- added JP1, JP2, JP3, JP4: Jumper_2_Open, Jumper:SolderJumper-2_P1.3mm_Open_RoundedPad1.0x1.5mm, symbol Jumper:Jumper_2_Open
- added Q1, Q2, Q3, Q4: 2N7002, Package_DFN_QFN:Diodes_DFN1006-3, symbol Transistor_FET:2N7002
- added TP6, TP7: TestPoint, TestPoint:TestPoint_Pad_D1.0mm, symbol Connector:TestPoint
- R10, R16, R21: value 1k -> 10k
- R14, R20, R9: value 0R -> 1k; now fitted
- R15: value 0R -> 10k; now fitted
Connections:
- net +3V3: now also R14.2, R19.2, R20.2, R9.2; no longer R14.1, R15.1, R20.1, R9.1
- net CAN0_RES: now also R15.1, Q1.1 (G); no longer R19.2
- net CAN1_RES: now also R10.1, Q2.1 (G); no longer R10.2
- net CAN2_RES: now also R16.1, Q3.1 (G); no longer R16.2
- net CAN3_RES: now also R21.1, Q4.1 (G); no longer R21.2
- net DBG_RX: now also TP6.1
- net DBG_TX: now also TP7.1
- net GND: now also R10.2, R15.2, R16.2, R21.2, JP1.2 (B), JP2.2 (B), JP3.2 (B), JP4.2 (B), Q1.2 (S), Q2.2 (S), Q3.2 (S), Q4.2 (S); no longer U10.2, U12.2, U7.1, U9.2
- net at R19.1, U9.1: no longer R15.2
- net at D10.2 (A2), FL1.3, J3.2 (Pin_2): now also U9.4; no longer U9.3
- net at R11.1: now also U9.3; no longer U9.4
- new net: JP4.1 (A), Q4.3 (D), U12.2
- new net: JP1.1 (A), Q1.3 (D), U9.2
- new net: R20.1, U12.1
- new net: R9.1, U7.1
- new net: JP2.1 (A), Q2.3 (D), U7.2
- new net: R14.1, U10.1
- new net: JP3.1 (A), Q3.3 (D), U10.2
Other:
- moved on the sheet: U9

Commit message: release: v1.1.0
Parts:
- added D14: LED_G, LED_SMD:LED_0603_1608Metric, symbol Device:LED
- added R23: 5.1k, Resistor_SMD:R_0402_1005Metric, symbol Device:R
Connections:
- net GND: now also D14.1 (K)
- net SYS: now reaches U2.25 (PB10/TMR0.COMP2/URT2.DE/URT2.RTS/SPI2.CS0/CAN2.STBY/ACMP.COMP0/USB0.PWR/ADC0.IN2/ADC1.IN2/CMP0.INP4/CMP1.INP4)
- net SYS: now also R23.1
- net at D8.2 (DOUT): now also D3.4 (DIN)
- net RGB_R: no longer names the net of U2.22 (PB13/TMR1.COMP3/URT3.DE/URT3.RTS/I2C3.SCL/SPI2.MOSI/CAN3.STBY/TRGM0.P01/ADC0.IN5/ADC1.IN5/CMP0.INP2/CMP1.INP2)
- net RGB_R: no longer D3.4 (DIN)
- new net: D14.2 (A), R23.2
- no-connect marks 12 -> 11
